Commit message: robot + field update

File: catchrobo_description/robots/catchrobo.urdf.xacro (robot description, xacro)
@@ -5,5 +5,4 @@
   <xacro:property name="field" value="$(arg field)" />
   <!-- Dependencies -->
-  <xacro:include filename="$(find catchrobo_description)/urdf/materials.xacro" />
   <xacro:include filename="$(find catchrobo_description)/urdf/common.xacro" />
   <xacro:include filename="$(find catchrobo_description)/urdf/base.urdf.xacro" />

File: catchrobo_description/urdf/arm.urdf.xacro (robot description, xacro)
@@ -47,5 +47,5 @@
       <parent link="${prefix}arm/link1"/>
       <child link="${prefix}arm/link2_1"/>
-      <origin xyz="0 0.1035 0" rpy="0 ${-90*M_PI/180} ${180*M_PI/180}"/>
+      <origin xyz="0 0.1135 0" rpy="0 ${-90*M_PI/180} ${180*M_PI/180}"/>
       <axis xyz="0 0 1"/>
       <limit lower="-0.43925" upper="0.43925" effort="10" velocity="5" acceleration="5"/>
@@ -67,5 +67,5 @@
       <parent link="${prefix}arm/link2_1"/>
       <child link="${prefix}arm/link2_2"/>
-      <origin xyz="0.0422 0 0" rpy="0 0 0"/>
+      <origin xyz="0.044 0 0" rpy="0 0 0"/>
       <axis xyz="0 0 1"/>
       <limit lower="-0.43925" upper="${0.43925*2}" effort="10" velocity="5" acceleration="5"/>
@@ -88,5 +88,5 @@
       <parent link="${prefix}arm/link2_2"/>
       <child link="${prefix}arm/link3"/>
-      <origin xyz="0.025 0 -0.0095" rpy="${90*M_PI/180} 0 0"/>
+      <origin xyz="0.0266 0 -0.0095" rpy="${90*M_PI/180} 0 0"/>
       <axis xyz="0 0 1"/>
       <limit lower="0" upper="0.145" effort="10" velocity="5" acceleration="5"/>

File: catchrobo_description/urdf/base.urdf.xacro (robot description, xacro)
@@ -17,5 +17,5 @@
       <visual>
         <geometry>
-          <mesh filename="package://catchrobo_description/mesh/base/DAE/base.dae" scale="${visual_mesh_scale}"/>
+          <mesh filename="package://catchrobo_description/mesh/base/DAE/base_full.dae" scale="${visual_mesh_scale}"/>
         </geometry>
         <material name="white"/>
@@ -23,5 +23,5 @@
       <collision>
         <geometry>
-          <mesh filename="package://catchrobo_description/mesh/base/STL/base.stl" scale="${collision_mesh_scale}"/>
+          <mesh filename="package://catchrobo_description/mesh/base/STL/base_full.stl" scale="${collision_mesh_scale}"/>
         </geometry>
       </collision>

File: catchrobo_description/urdf/gripper.urdf.xacro (robot description, xacro)
@@ -27,5 +27,5 @@
       <parent link="${prefix}gripper/base_link"/>
       <child link="${prefix}gripper/left_finger"/>
-      <origin xyz="0.2438 0.0365 -0.076" rpy="${90*M_PI/180} 0 ${90*M_PI/180}"/>
+      <origin xyz="0.2511 0.0365 -0.086" rpy="${90*M_PI/180} 0 ${90*M_PI/180}"/>
       <axis xyz="0 0 1"/>
       <limit lower="${0*M_PI/180}" upper="${90*M_PI/180}" effort="6"
@@ -48,5 +48,5 @@
       <parent link="${prefix}gripper/base_link"/>
       <child link="${prefix}gripper/right_finger"/>
-      <origin xyz="0.2438 -0.0365 -0.076" rpy="${90*M_PI/180} 0 ${90*M_PI/180}"/>
+      <origin xyz="0.2511 -0.0365 -0.086" rpy="${90*M_PI/180} 0 ${90*M_PI/180}"/>
       <axis xyz="0 0 1"/>
       <limit lower="${0*M_PI/180}" upper="${90*M_PI/180}" effort="6"
