Commit message: grasping_frameの位置を修正

File: catchrobo_description/urdf/gripper.urdf.xacro (robot description, xacro)
@@ -70,5 +70,5 @@
       <parent link="${prefix}gripper/base_link"/>
       <child link="${prefix}gripper/grasping_frame"/>
-      <origin xyz="0 0 0.1" rpy="0 0 0"/>
+      <origin xyz="0.2511 0 -0.1" rpy="0 0 0"/>
     </joint>
     <link name="${prefix}gripper/grasping_frame"/>
