Commit message: update

File: catchrobo_description/urdf/arm.urdf.xacro (robot description, xacro)
@@ -108,5 +108,5 @@
       <parent link="${prefix}arm/link3"/>
       <child link="${prefix}arm/link_tip"/>
-      <origin xyz="0 0 -0.1" rpy="${180*M_PI/180} 0 0"/>
+      <origin xyz="0.15 0 0" rpy="${180*M_PI/180} 0 0"/>
     </joint>
     <link name="${prefix}arm/link_tip"/>

File: catchrobo_description/urdf/base.urdf.xacro (robot description, xacro)
@@ -31,8 +31,8 @@
       <child link="base/link_tip"/>
       <xacro:if value="${field=='blue'}">
-        <origin xyz="-0.795 0.350 0.0044" rpy="0 0 0"/>
+        <origin xyz="-0.3 -0.825 0.00445" rpy="0 0 0"/>
       </xacro:if>
       <xacro:if value="${field=='red'}">
-        <origin xyz="0.795 0.350 0.0044" rpy="0 0 0"/>
+        <origin xyz="-0.3 0.825 0.00445" rpy="0 0 0"/>
       </xacro:if>
     </joint>

File: catchrobo_description/urdf/gripper.urdf.xacro (robot description, xacro)
@@ -27,5 +27,5 @@
       <parent link="${prefix}gripper/base_link"/>
       <child link="${prefix}gripper/finger1"/>
-      <origin xyz="0.1 0 0.05" rpy="0 0 0"/>
+      <origin xyz="0.05 0 0" rpy="0 0 ${90*M_PI/180}"/>
       <axis xyz="0 0 1"/>
       <limit lower="${0*M_PI/180}" upper="${90*M_PI/180}" effort="6"
@@ -48,5 +48,5 @@
       <parent link="${prefix}gripper/base_link"/>
       <child link="${prefix}gripper/finger2"/>
-      <origin xyz="0 -0.05 0.05" rpy="0 0 0"/>
+      <origin xyz="-0.025 -0.0433012 0" rpy="0 0 ${-30*M_PI/180}"/>
       <axis xyz="0 0 1"/>
       <limit lower="${0*M_PI/180}" upper="${90*M_PI/180}" effort="6"
@@ -70,5 +70,5 @@
       <parent link="${prefix}gripper/base_link"/>
       <child link="${prefix}gripper/finger3"/>
-      <origin xyz="0 0.05 0.05" rpy="0 0 0"/>
+      <origin xyz="-0.025 0.0433012 0" rpy="0 0 ${210*M_PI/180}"/>
       <axis xyz="0 0 1"/>
       <limit lower="${0*M_PI/180}" upper="${90*M_PI/180}" effort="6"

Commit message: gazebo not work

File: catchrobo_description/urdf/arm.urdf.xacro (robot description, xacro)
@@ -1,4 +1,6 @@
 <?xml version="1.0"?>
 <robot xmlns:xacro="http://ros.org/wiki/xacro">
+    <xacro:include filename="$(find catchrobo_description)/urdf/arm.transmission.xacro"/>
+  <xacro:include filename="$(find catchrobo_description)/urdf/arm.gazebo.xacro"/>
   <!-- Constants -->
   <xacro:property name="visual_mesh_scale" value="1.0 1.0 1.0"/>
@@ -23,4 +25,11 @@
         </geometry>
       </collision>
+    <inertial>
+      <origin xyz="0 0 0.013" rpy="0 0 0"/>
+      <mass value="0.25"/>
+      <inertia ixx="0.0003350833" ixy="0" ixz="0"
+        iyy="0.000560417" iyz="0"
+        izz="0.000478833"/>
+    </inertial>
     </link>
     <joint name="${prefix}arm/joint1" type="prismatic">
@@ -43,4 +52,11 @@
         </geometry>
       </collision>
+    <inertial>
+      <origin xyz="0 0 0.013" rpy="0 0 0"/>
+      <mass value="0.25"/>
+      <inertia ixx="0.0003350833" ixy="0" ixz="0"
+        iyy="0.000560417" iyz="0"
+        izz="0.000478833"/>
+    </inertial>
     </link>
     <joint name="${prefix}arm/joint2" type="prismatic">
@@ -63,4 +79,11 @@
         </geometry>
       </collision>
+          <inertial>
+      <origin xyz="0 0 0.013" rpy="0 0 0"/>
+      <mass value="0.25"/>
+      <inertia ixx="0.0003350833" ixy="0" ixz="0"
+        iyy="0.000560417" iyz="0"
+        izz="0.000478833"/>
+    </inertial>
     </link>
     <joint name="${prefix}arm/joint2_mimic" type="prismatic">
@@ -84,4 +107,11 @@
         </geometry>
       </collision>
+          <inertial>
+      <origin xyz="0 0 0.013" rpy="0 0 0"/>
+      <mass value="0.25"/>
+      <inertia ixx="0.0003350833" ixy="0" ixz="0"
+        iyy="0.000560417" iyz="0"
+        izz="0.000478833"/>
+    </inertial>
     </link>
     <joint name="${prefix}arm/joint3" type="prismatic">
@@ -104,4 +134,11 @@
         </geometry>
       </collision>
+          <inertial>
+      <origin xyz="0 0 0.013" rpy="0 0 0"/>
+      <mass value="0.25"/>
+      <inertia ixx="0.0003350833" ixy="0" ixz="0"
+        iyy="0.000560417" iyz="0"
+        izz="0.000478833"/>
+    </inertial>
     </link>
     <joint name="${prefix}arm/joint_tip" type="fixed">

File: catchrobo_description/urdf/base.urdf.xacro (robot description, xacro)
@@ -1,4 +1,5 @@
 <?xml version="1.0"?>
 <robot xmlns:xacro="http://ros.org/wiki/xacro">
+  <xacro:include filename="$(find catchrobo_description)/urdf/base.gazebo.xacro"/>
   <!-- Field Side Parameters-->
   <xacro:arg name="field" default=""/>
@@ -26,4 +27,11 @@
         </geometry>
       </collision>
+    <inertial>
+      <origin xyz="0 0 0.013" rpy="0 0 0"/>
+      <mass value="0.25"/>
+      <inertia ixx="0.0003350833" ixy="0" ixz="0"
+        iyy="0.000560417" iyz="0"
+        izz="0.000478833"/>
+    </inertial>
     </link>
     <joint name="base/link_tip" type="fixed">

File: catchrobo_description/urdf/gripper.urdf.xacro (robot description, xacro)
@@ -23,4 +23,11 @@
         </geometry>
       </collision>
+    <inertial>
+      <origin xyz="0 0 0.013" rpy="0 0 0"/>
+      <mass value="0.25"/>
+      <inertia ixx="0.0003350833" ixy="0" ixz="0"
+        iyy="0.000560417" iyz="0"
+        izz="0.000478833"/>
+    </inertial>
     </link>
     <joint name="${prefix}gripper/joint1" type="revolute">
@@ -44,4 +51,11 @@
         </geometry>
       </collision>
+          <inertial>
+      <origin xyz="0 0 0.013" rpy="0 0 0"/>
+      <mass value="0.25"/>
+      <inertia ixx="0.0003350833" ixy="0" ixz="0"
+        iyy="0.000560417" iyz="0"
+        izz="0.000478833"/>
+    </inertial>
     </link>
     <joint name="${prefix}gripper/joint2" type="revolute">
@@ -66,4 +80,11 @@
         </geometry>
       </collision>
+          <inertial>
+      <origin xyz="0 0 0.013" rpy="0 0 0"/>
+      <mass value="0.25"/>
+      <inertia ixx="0.0003350833" ixy="0" ixz="0"
+        iyy="0.000560417" iyz="0"
+        izz="0.000478833"/>
+    </inertial>
     </link>
     <joint name="${prefix}gripper/joint3" type="revolute">
@@ -88,4 +109,11 @@
         </geometry>
       </collision>
+          <inertial>
+      <origin xyz="0 0 0.013" rpy="0 0 0"/>
+      <mass value="0.25"/>
+      <inertia ixx="0.0003350833" ixy="0" ixz="0"
+        iyy="0.000560417" iyz="0"
+        izz="0.000478833"/>
+    </inertial>
     </link>
     <joint name="${prefix}gripper/grasping_frame_joint" type="fixed">

Commit message: mesh, urdfを更新

File: catchrobo_description/urdf/arm.urdf.xacro (robot description, xacro)
@@ -14,5 +14,5 @@
       <visual>
         <geometry>
-          <mesh filename="package://catchrobo_description/mesh/arm/visual/link0.stl" scale="${visual_mesh_scale}"/>
+          <mesh filename="package://catchrobo_description/mesh/arm/DAE/link0.dae" scale="${visual_mesh_scale}"/>
         </geometry>
         <material name="white"/>
@@ -20,5 +20,5 @@
       <collision>
         <geometry>
-          <mesh filename="package://catchrobo_description/mesh/arm/collision/link0.stl" scale="${collision_mesh_scale}"/>
+          <mesh filename="package://catchrobo_description/mesh/arm/STL/link0.stl" scale="${collision_mesh_scale}"/>
         </geometry>
       </collision>
@@ -27,12 +27,12 @@
       <parent link="${prefix}arm/link0"/>
       <child link="${prefix}arm/link1"/>
-      <origin xyz="0 0 0.1" rpy="0 ${90*M_PI/180} 0"/>
+      <origin xyz="-0.90625 0 0.0485" rpy="${90*M_PI/180} 0 ${90*M_PI/180}"/>
       <axis xyz="0 0 1"/>
-      <limit lower="0" upper="1.5" effort="10" velocity="5" acceleration="5"/>
+      <limit lower="0" upper="1.3525" effort="10" velocity="5" acceleration="5"/>
     </joint>
     <link name="${prefix}arm/link1">
       <visual>
         <geometry>
-          <mesh filename="package://catchrobo_description/mesh/arm/visual/link1.stl" scale="${visual_mesh_scale}"/>
+          <mesh filename="package://catchrobo_description/mesh/arm/DAE/link1.dae" scale="${visual_mesh_scale}"/>
         </geometry>
         <material name="white"/>
@@ -40,5 +40,5 @@
       <collision>
         <geometry>
-          <mesh filename="package://catchrobo_description/mesh/arm/collision/link1.stl" scale="${collision_mesh_scale}"/>
+          <mesh filename="package://catchrobo_description/mesh/arm/STL/link1.stl" scale="${collision_mesh_scale}"/>
         </geometry>
       </collision>
@@ -47,12 +47,12 @@
       <parent link="${prefix}arm/link1"/>
       <child link="${prefix}arm/link2_1"/>
-      <origin xyz="-0.1 0 0" rpy="${-90*M_PI/180} 0 0"/>
+      <origin xyz="0 0.1035 0" rpy="0 ${-90*M_PI/180} ${180*M_PI/180}"/>
       <axis xyz="0 0 1"/>
-      <limit lower="-0.5" upper="0.5" effort="10" velocity="5" acceleration="5"/>
+      <limit lower="-0.43925" upper="0.43925" effort="10" velocity="5" acceleration="5"/>
     </joint>
     <link name="${prefix}arm/link2_1">
       <visual>
         <geometry>
-          <mesh filename="package://catchrobo_description/mesh/arm/visual/link2_1.stl" scale="${visual_mesh_scale}"/>
+          <mesh filename="package://catchrobo_description/mesh/arm/DAE/link2_1.dae" scale="${visual_mesh_scale}"/>
         </geometry>
         <material name="white"/>
@@ -60,5 +60,5 @@
       <collision>
         <geometry>
-          <mesh filename="package://catchrobo_description/mesh/arm/collision/link2_1.stl" scale="${collision_mesh_scale}"/>
+          <mesh filename="package://catchrobo_description/mesh/arm/STL/link2_1.stl" scale="${collision_mesh_scale}"/>
         </geometry>
       </collision>
@@ -67,7 +67,7 @@
       <parent link="${prefix}arm/link2_1"/>
       <child link="${prefix}arm/link2_2"/>
-      <origin xyz="0 -0.1 0" rpy="0 0 0"/>
+      <origin xyz="0.0422 0 0" rpy="0 0 0"/>
       <axis xyz="0 0 1"/>
-      <limit lower="0" upper="1" effort="10" velocity="5" acceleration="5"/>
+      <limit lower="-0.43925" upper="${0.43925*2}" effort="10" velocity="5" acceleration="5"/>
        <mimic joint="${prefix}arm/joint2" multiplier="1" offset="0" />
     </joint>
@@ -75,5 +75,5 @@
       <visual>
         <geometry>
-          <mesh filename="package://catchrobo_description/mesh/arm/visual/link2_2.stl" scale="${visual_mesh_scale}"/>
+          <mesh filename="package://catchrobo_description/mesh/arm/DAE/link2_2.dae" scale="${visual_mesh_scale}"/>
         </geometry>
         <material name="white"/>
@@ -81,5 +81,5 @@
       <collision>
         <geometry>
-          <mesh filename="package://catchrobo_description/mesh/arm/collision/link2_2.stl" scale="${collision_mesh_scale}"/>
+          <mesh filename="package://catchrobo_description/mesh/arm/STL/link2_2.stl" scale="${collision_mesh_scale}"/>
         </geometry>
       </collision>
@@ -88,12 +88,12 @@
       <parent link="${prefix}arm/link2_2"/>
       <child link="${prefix}arm/link3"/>
-      <origin xyz="0 -0.1 0" rpy="${90*M_PI/180} 0 ${-90*M_PI/180}"/>
+      <origin xyz="0.025 0 -0.0095" rpy="${90*M_PI/180} 0 0"/>
       <axis xyz="0 0 1"/>
-      <limit lower="0" upper="0.3" effort="10" velocity="5" acceleration="5"/>
+      <limit lower="0" upper="0.145" effort="10" velocity="5" acceleration="5"/>
     </joint>
     <link name="${prefix}arm/link3">
       <visual>
         <geometry>
-          <mesh filename="package://catchrobo_description/mesh/arm/visual/link3.stl" scale="${visual_mesh_scale}"/>
+          <mesh filename="package://catchrobo_description/mesh/arm/DAE/link3.dae" scale="${visual_mesh_scale}"/>
         </geometry>
         <material name="white"/>
@@ -101,5 +101,5 @@
       <collision>
         <geometry>
-          <mesh filename="package://catchrobo_description/mesh/arm/collision/link3.stl" scale="${collision_mesh_scale}"/>
+          <mesh filename="package://catchrobo_description/mesh/arm/STL/link3.stl" scale="${collision_mesh_scale}"/>
         </geometry>
       </collision>
@@ -108,5 +108,5 @@
       <parent link="${prefix}arm/link3"/>
       <child link="${prefix}arm/link_tip"/>
-      <origin xyz="0.15 0 0" rpy="${180*M_PI/180} 0 0"/>
+      <origin xyz="0 0 0" rpy="0 0 0"/>
     </joint>
     <link name="${prefix}arm/link_tip"/>

File: catchrobo_description/urdf/base.urdf.xacro (robot description, xacro)
@@ -17,5 +17,5 @@
       <visual>
         <geometry>
-          <mesh filename="package://catchrobo_description/mesh/base/visual/base.dae" scale="${visual_mesh_scale}"/>
+          <mesh filename="package://catchrobo_description/mesh/base/DAE/base.dae" scale="${visual_mesh_scale}"/>
         </geometry>
         <material name="white"/>
@@ -23,5 +23,5 @@
       <collision>
         <geometry>
-          <mesh filename="package://catchrobo_description/mesh/base/collision/base.stl" scale="${collision_mesh_scale}"/>
+          <mesh filename="package://catchrobo_description/mesh/base/STL/base.stl" scale="${collision_mesh_scale}"/>
         </geometry>
       </collision>
@@ -31,8 +31,8 @@
       <child link="base/link_tip"/>
       <xacro:if value="${field=='blue'}">
-        <origin xyz="-0.3 -0.825 0.00445" rpy="0 0 0"/>
+        <origin xyz="0.675 -0.825 0.00445" rpy="0 0 0"/>
       </xacro:if>
       <xacro:if value="${field=='red'}">
-        <origin xyz="-0.3 0.825 0.00445" rpy="0 0 0"/>
+        <origin xyz="0.675 0.825 0.00445" rpy="0 0 0"/>
       </xacro:if>
     </joint>

File: catchrobo_description/urdf/gripper.urdf.xacro (robot description, xacro)
@@ -14,5 +14,5 @@
       <visual>
         <geometry>
-          <mesh filename="package://catchrobo_description/mesh/gripper/visual/base.stl" scale="${visual_mesh_scale}"/>
+          <mesh filename="package://catchrobo_description/mesh/gripper/DAE/base.dae" scale="${visual_mesh_scale}"/>
         </geometry>
         <material name="white"/>
@@ -20,5 +20,5 @@
       <collision>
         <geometry>
-          <mesh filename="package://catchrobo_description/mesh/gripper/collision/base.stl" scale="${collision_mesh_scale}"/>
+          <mesh filename="package://catchrobo_description/mesh/gripper/STL/base.stl" scale="${collision_mesh_scale}"/>
         </geometry>
       </collision>
@@ -26,14 +26,14 @@
     <joint name="${prefix}gripper/joint1" type="revolute">
       <parent link="${prefix}gripper/base_link"/>
-      <child link="${prefix}gripper/finger1"/>
-      <origin xyz="0.05 0 0" rpy="0 0 ${90*M_PI/180}"/>
+      <child link="${prefix}gripper/left_finger"/>
+      <origin xyz="0.2438 0.0365 -0.076" rpy="${90*M_PI/180} 0 ${90*M_PI/180}"/>
       <axis xyz="0 0 1"/>
       <limit lower="${0*M_PI/180}" upper="${90*M_PI/180}" effort="6"
               velocity="5" acceleration="5"/>
     </joint>
-    <link name="${prefix}gripper/finger1">
+    <link name="${prefix}gripper/left_finger">
       <visual>
         <geometry>
-          <mesh filename="package://catchrobo_description/mesh/gripper/visual/finger.stl" scale="${visual_mesh_scale}"/>
+          <mesh filename="package://catchrobo_description/mesh/gripper/DAE/left_finger.dae" scale="${visual_mesh_scale}"/>
         </geometry>
         <material name="orange"/>
@@ -41,21 +41,21 @@
       <collision>
         <geometry>
-          <mesh filename="package://catchrobo_description/mesh/gripper/collision/finger.stl" scale="${collision_mesh_scale}"/>
+          <mesh filename="package://catchrobo_description/mesh/gripper/STL/left_finger.stl" scale="${collision_mesh_scale}"/>
         </geometry>
       </collision>
     </link>
-    <joint name="${prefix}gripper/joint2" type="revolute">
+    <joint name="${prefix}gripper/joint1_mimic" type="revolute">
       <parent link="${prefix}gripper/base_link"/>
-      <child link="${prefix}gripper/finger2"/>
-      <origin xyz="-0.025 -0.0433012 0" rpy="0 0 ${-30*M_PI/180}"/>
+      <child link="${prefix}gripper/right_finger"/>
+      <origin xyz="0.2438 -0.0365 -0.076" rpy="${90*M_PI/180} 0 ${90*M_PI/180}"/>
       <axis xyz="0 0 1"/>
       <limit lower="${0*M_PI/180}" upper="${90*M_PI/180}" effort="6"
               velocity="5" acceleration="5"/>
-      <mimic joint="${prefix}gripper/joint1" multiplier="1" offset="0" />
+      <mimic joint="${prefix}gripper/joint1" multiplier="-1" offset="0" />
     </joint>
-    <link name="${prefix}gripper/finger2">
+    <link name="${prefix}gripper/right_finger">
       <visual>
         <geometry>
-          <mesh filename="package://catchrobo_description/mesh/gripper/visual/finger.stl" scale="${visual_mesh_scale}"/>
+          <mesh filename="package://catchrobo_description/mesh/gripper/DAE/right_finger.dae" scale="${visual_mesh_scale}"/>
         </geometry>
         <material name="orange"/>
@@ -63,27 +63,5 @@
       <collision>
         <geometry>
-          <mesh filename="package://catchrobo_description/mesh/gripper/collision/finger.stl" scale="${collision_mesh_scale}"/>
-        </geometry>
-      </collision>
-    </link>
-    <joint name="${prefix}gripper/joint3" type="revolute">
-      <parent link="${prefix}gripper/base_link"/>
-      <child link="${prefix}gripper/finger3"/>
-      <origin xyz="-0.025 0.0433012 0" rpy="0 0 ${210*M_PI/180}"/>
-      <axis xyz="0 0 1"/>
-      <limit lower="${0*M_PI/180}" upper="${90*M_PI/180}" effort="6"
-              velocity="5" acceleration="5"/>
-      <mimic joint="${prefix}gripper/joint1" multiplier="1" offset="0" />
-    </joint>
-    <link name="${prefix}gripper/finger3">
-      <visual>
-        <geometry>
-          <mesh filename="package://catchrobo_description/mesh/gripper/visual/finger.stl" scale="${visual_mesh_scale}"/>
-        </geometry>
-        <material name="orange"/>
-      </visual>
-      <collision>
-        <geometry>
-          <mesh filename="package://catchrobo_description/mesh/gripper/collision/finger.stl" scale="${collision_mesh_scale}"/>
+          <mesh filename="package://catchrobo_description/mesh/gripper/STL/right_finger.stl" scale="${collision_mesh_scale}"/>
         </geometry>
       </collision>

Commit message: Link2位置修正

File: catchrobo_description/urdf/arm.urdf.xacro (robot description, xacro)
@@ -67,5 +67,5 @@
       <parent link="${prefix}arm/link2_1"/>
       <child link="${prefix}arm/link2_2"/>
-      <origin xyz="0.044 0 0" rpy="0 0 0"/>
+      <origin xyz="0.041 0 0" rpy="0 0 0"/>
       <axis xyz="0 0 1"/>
       <limit lower="-0.43925" upper="${0.43925*2}" effort="10" velocity="5" acceleration="5"/>
@@ -88,5 +88,5 @@
       <parent link="${prefix}arm/link2_2"/>
       <child link="${prefix}arm/link3"/>
-      <origin xyz="0.0266 0 -0.0095" rpy="${90*M_PI/180} 0 0"/>
+      <origin xyz="0.0296 0 0" rpy="${90*M_PI/180} 0 0"/>
       <axis xyz="0 0 1"/>
       <limit lower="0" upper="0.145" effort="10" velocity="5" acceleration="5"/>

Commit message: J3の原点ズレを修正

File: catchrobo_description/urdf/arm.urdf.xacro (robot description, xacro)
@@ -88,5 +88,5 @@
       <parent link="${prefix}arm/link2_2"/>
       <child link="${prefix}arm/link3"/>
-      <origin xyz="0.0296 0 0" rpy="${90*M_PI/180} 0 0"/>
+      <origin xyz="0.0296 -0.01 0" rpy="${90*M_PI/180} 0 0"/>
       <axis xyz="0 0 1"/>
       <limit lower="0" upper="0.145" effort="10" velocity="5" acceleration="5"/>

Commit message: URDFのmaterialタグを削除

File: catchrobo_description/urdf/arm.urdf.xacro (robot description, xacro)
@@ -16,5 +16,4 @@
           <mesh filename="package://catchrobo_description/mesh/arm/DAE/link0.dae" scale="${visual_mesh_scale}"/>
         </geometry>
-        <material name="white"/>
       </visual>
       <collision>
@@ -36,5 +35,4 @@
           <mesh filename="package://catchrobo_description/mesh/arm/DAE/link1.dae" scale="${visual_mesh_scale}"/>
         </geometry>
-        <material name="white"/>
       </visual>
       <collision>
@@ -56,5 +54,4 @@
           <mesh filename="package://catchrobo_description/mesh/arm/DAE/link2_1.dae" scale="${visual_mesh_scale}"/>
         </geometry>
-        <material name="white"/>
       </visual>
       <collision>
@@ -77,5 +74,4 @@
           <mesh filename="package://catchrobo_description/mesh/arm/DAE/link2_2.dae" scale="${visual_mesh_scale}"/>
         </geometry>
-        <material name="white"/>
       </visual>
       <collision>
@@ -97,5 +93,4 @@
           <mesh filename="package://catchrobo_description/mesh/arm/DAE/link3.dae" scale="${visual_mesh_scale}"/>
         </geometry>
-        <material name="white"/>
       </visual>
       <collision>

File: catchrobo_description/urdf/base.urdf.xacro (robot description, xacro)
@@ -20,5 +20,4 @@
             <mesh filename="package://catchrobo_description/mesh/base/DAE/base_full_without_box_blue.dae" scale="${visual_mesh_scale}"/>
           </geometry>
-          <material name="white"/>
         </visual>
         <collision>
@@ -33,5 +32,4 @@
             <mesh filename="package://catchrobo_description/mesh/base/DAE/base_full_without_box_red.dae" scale="${visual_mesh_scale}"/>
           </geometry>
-          <material name="white"/>
         </visual>
         <collision>
@@ -68,5 +66,4 @@
           <mesh filename="package://catchrobo_description/mesh/base/DAE/box.dae" scale="${visual_mesh_scale}"/>
         </geometry>
-        <material name="white"/>
       </visual>
       <collision>

File: catchrobo_description/urdf/gripper.urdf.xacro (robot description, xacro)
@@ -16,5 +16,4 @@
           <mesh filename="package://catchrobo_description/mesh/gripper/DAE/base.dae" scale="${visual_mesh_scale}"/>
         </geometry>
-        <material name="white"/>
       </visual>
       <collision>
@@ -37,5 +36,4 @@
           <mesh filename="package://catchrobo_description/mesh/gripper/DAE/left_finger.dae" scale="${visual_mesh_scale}"/>
         </geometry>
-        <material name="orange"/>
       </visual>
       <collision>
@@ -59,5 +57,4 @@
           <mesh filename="package://catchrobo_description/mesh/gripper/DAE/right_finger.dae" scale="${visual_mesh_scale}"/>
         </geometry>
-        <material name="orange"/>
       </visual>
       <collision>
